File: OBC.kicad_sch (KiCad schematic)
At the start: 20 parts, among them J1 BOOTSEL, J2 10118194-0001LF, J3 DF40C-70DP-0.4V_51_, J4 DF40C-70DP-0.4V_51_, J5 DF40C-70DP-0.4V_51_, U1 W25Q16JVUXIQ TR, U2 LTC2854HDD-PBF

Commit message: Initial schematic entry
Parts:
- removed A1: ~, ODYSSEY-STM32MP157C-SOM:ODYSSEY-STM32MP157C-SOM, symbol ODYSSEY-STM32MP157C-SOM:ODYSSEY-STM32MP157C-SOM
- removed C1: 100n, Capacitor_SMD:C_0603_1608Metric, symbol Device:C_Small
- removed C2: 2u2, Capacitor_SMD:C_0603_1608Metric, symbol Device:C_Small
- removed J1: BOOTSEL, Connector_PinHeader_2.54mm:PinHeader_1x02_P2.54mm_Horizontal, symbol Connector_Generic:Conn_01x02
- removed J2: 10118194-0001LF, 10118194_0001LF:AMPHENOL_10118194-0001LF, symbol 10118194-0001LF:10118194-0001LF
- removed J3, J4, J5: DF40C-70DP-0.4V_51_, DF40C-70DP-0.4V_51_:HIROSE_DF40C-70DP-0.4V_51_, symbol DF40C-70DP-0.4V_51_:DF40C-70DP-0.4V_51_
- removed R1: 1k, Resistor_SMD:R_0603_1608Metric, symbol Device:R_Small_US
- removed U1: W25Q16JVUXIQ TR, W25Q16JVUXIQ:USON-8_UX_2x3x0p6_WIN, symbol 2024-12-07_14-34-38:W25Q16JVUXIQ_TR
- added D2: LED Green, LED_SMD:LED_0603_1608Metric, symbol Device:LED
- added J3: Conn_01x03, Connector_PinHeader_2.54mm:PinHeader_1x03_P2.54mm_Vertical, symbol Connector_Generic:Conn_01x03
- added Module1: ComputeModule4, CM4IO:Raspberry-Pi-4-Compute-Module, symbol CM4IO:ComputeModule4-CM4
- added R1: 1k, Resistor_SMD:R_0402_1005Metric, symbol Device:R
- added TP3: TestPoint, TestPoint:TestPoint_Pad_2.0x2.0mm, symbol Connector:TestPoint
Connections:
- net GND: now also J3.2 (Pin_2), Module1.1 (GND), Module1.107 (GND), Module1.108 (GND), Module1.113 (GND), Module1.114 (GND), Module1.119 (GND), Module1.120 (GND), Module1.125 (GND), Module1.126 (GND), Module1.13 (GND), Module1.131 (GND), Module1.132 (GND), Module1.137 (GND), Module1.138 (GND), Module1.14 (GND), Module1.144 (GND), Module1.150 (GND), Module1.155 (GND), Module1.156 (GND), Module1.161 (GND), Module1.162 (GND), Module1.167 (GND), Module1.168 (GND), Module1.173 (GND), Module1.174 (GND), Module1.179 (GND), Module1.180 (GND), Module1.185 (GND), Module1.186 (GND), Module1.191 (GND), Module1.192 (GND), Module1.197 (GND), Module1.198 (GND), Module1.2 (GND), Module1.22 (GND), Module1.23 (GND), Module1.32 (GND), Module1.33 (GND), Module1.42 (GND), Module1.43 (GND), Module1.52 (GND), Module1.53 (GND), Module1.59 (GND), Module1.60 (GND), Module1.65 (GND), Module1.66 (GND), Module1.7 (GND), Module1.71 (GND), Module1.74 (GND), Module1.8 (GND), Module1.98 (GND)
- net SCL0: now also Module1.80 (SCL0)
- net SDA0: now also Module1.82 (SDA0)
- net BUS5V: now reaches H2.25
- net BUS5V: now also H2.26
- new net: D2.1 (K), R1.1, TP3.1
- new net: Module1.21 (PI_nLED_Activity), R1.2
- new net +1.8v: Module1.88 (+1.8v_(Output)), Module1.90 (+1.8v_(Output))
- new net +3.3v: D2.2 (A), Module1.84 (+3.3v_(Output)), Module1.86 (+3.3v_(Output))
- new net +5v: Module1.77 (+5v_(Input)), Module1.79 (+5v_(Input)), Module1.81 (+5v_(Input)), Module1.83 (+5v_(Input)), Module1.85 (+5v_(Input)), Module1.87 (+5v_(Input))
- new net AIN0: Module1.96 (AnalogIP1)
- new net AIN1: Module1.94 (AnalogIP0)
- new net BT_nDis: J3.3 (Pin_3), Module1.91 (BT_nDisable)
- new net CAM0_C_N: Module1.140 (CAM0_C_N)
- new net CAM0_C_P: Module1.142 (CAM0_C_P)
- new net CAM0_D0_N: Module1.128 (CAM0_D0_N)
- new net CAM0_D0_P: Module1.130 (CAM0_D0_P)
- new net CAM0_D1_N: Module1.134 (CAM0_D1_N)
- new net CAM0_D1_P: Module1.136 (CAM0_D1_P)
- new net CAM1_C_N: Module1.127 (CAM1_C_N)
- new net CAM1_C_P: Module1.129 (CAM1_C_P)
- new net CAM1_D0_N: Module1.115 (CAM1_D0_N)
- new net CAM1_D0_P: Module1.117 (CAM1_D0_P)
- new net CAM1_D1_N: Module1.121 (CAM1_D1_N)
- new net CAM1_D1_P: Module1.123 (CAM1_D1_P)
- new net CAM1_D2_N: Module1.133 (CAM1_D2_N)
- new net CAM1_D2_P: Module1.135 (CAM1_D2_P)
- new net CAM1_D3_N: Module1.139 (CAM1_D3_N)
- new net CAM1_D3_P: Module1.141 (CAM1_D3_P)
- new net CAM_GPIO: Module1.97 (Camera_GPIO)
- new net DSI0_C_N: Module1.169 (DSI0_C_N)
- new net DSI0_C_P: Module1.171 (DSI0_C_P)
- new net DSI0_D0_N: Module1.157 (DSI0_D0_N)
- new net DSI0_D0_P: Module1.159 (DSI0_D0_P)
- new net DSI0_D1_N: Module1.163 (DSI0_D1_N)
- new net DSI0_D1_P: Module1.165 (DSI0_D1_P)
- new net DSI1_C_N: Module1.187 (DSI1_C_N)
- new net DSI1_C_P: Module1.189 (DSI1_C_P)
- new net DSI1_D0_N: Module1.175 (DSI1_D0_N)
- new net DSI1_D0_P: Module1.177 (DSI1_D0_P)
- new net DSI1_D1_N: Module1.181 (DSI1_D1_N)
- new net DSI1_D1_P: Module1.183 (DSI1_D1_P)
- new net DSI1_D2_N: Module1.193 (DSI1_D2_N)
- new net DSI1_D2_P: Module1.195 (DSI1_D2_P)
- new net DSI1_D3_N: Module1.194 (DSI1_D3_N)
- new net DSI1_D3_P: Module1.196 (DSI1_D3_P)
- new net EEPROM_nWP: Module1.20 (EEPROM_nWP)
- new net ETH_LEDG: Module1.17 (Ethernet_nLED2(3.3v))
- new net ETH_LEDY: Module1.15 (Ethernet_nLED3(3.3v))
- new net GLOBAL_EN: Module1.99 (Global_EN)
- new net GPIO10: Module1.44 (GPIO10)
- new net GPIO11: Module1.38 (GPIO11)
- new net GPIO12: Module1.31 (GPIO12)
- new net GPIO13: Module1.28 (GPIO13)
- new net GPIO14: Module1.55 (GPIO14)
- new net GPIO15: Module1.51 (GPIO15)
- new net GPIO16: Module1.29 (GPIO16)
- new net GPIO17: Module1.50 (GPIO17)
- new net GPIO18: Module1.49 (GPIO18)
- new net GPIO19: Module1.26 (GPIO19)
- new net GPIO2: Module1.58 (GPIO2)
- new net GPIO20: Module1.27 (GPIO20)
- new net GPIO21: Module1.25 (GPIO21)
- new net GPIO22: Module1.46 (GPIO22)
- new net GPIO23: Module1.47 (GPIO23)
- new net GPIO24: Module1.45 (GPIO24)
- new net GPIO25: Module1.41 (GPIO25)
- new net GPIO26: Module1.24 (GPIO26)
- new net GPIO27: Module1.48 (GPIO27)
- new net GPIO3: Module1.56 (GPIO3)
- new net GPIO4: Module1.54 (GPIO4)
- new net GPIO5: Module1.34 (GPIO5)
- new net GPIO6: Module1.30 (GPIO6)
- new net GPIO7: Module1.37 (GPIO7)
- new net GPIO8: Module1.39 (GPIO8)
- new net GPIO9: Module1.40 (GPIO9)
- new net GPIO_VREF: Module1.78 (GPIO_VREF(1.8v/3.3v_Input))
- new net HDMI0_CEC: Module1.151 (HDMI0_CEC)
- new net HDMI0_CK_N: Module1.190 (HDMI0_CLK_N)
- new net HDMI0_CK_P: Module1.188 (HDMI0_CLK_P)
- new net HDMI0_D0_N: Module1.184 (HDMI0_TX0_N)
- new net HDMI0_D0_P: Module1.182 (HDMI0_TX0_P)
- new net HDMI0_D1_N: Module1.178 (HDMI0_TX1_N)
- new net HDMI0_D1_P: Module1.176 (HDMI0_TX1_P)
- new net HDMI0_D2_N: Module1.172 (HDMI0_TX2_N)
- new net HDMI0_D2_P: Module1.170 (HDMI0_TX2_P)
- new net HDMI0_HOTPLUG: Module1.153 (HDMI0_HOTPLUG)
- new net HDMI0_SCL: Module1.200 (HDMI0_SCL)
- new net HDMI0_SDA: Module1.199 (HDMI0_SDA)
- new net HDMI1_CEC: Module1.149 (HDMI1_CEC)
- new net HDMI1_CK_N: Module1.166 (HDMI1_CLK_N)
- new net HDMI1_CK_P: Module1.164 (HDMI1_CLK_P)
- new net HDMI1_D0_N: Module1.160 (HDMI1_TX0_N)
- new net HDMI1_D0_P: Module1.158 (HDMI1_TX0_P)
- new net HDMI1_D1_N: Module1.154 (HDMI1_TX1_N)
- new net HDMI1_D1_P: Module1.152 (HDMI1_TX1_P)
- new net HDMI1_D2_N: Module1.148 (HDMI1_TX2_N)
- new net HDMI1_D2_P: Module1.146 (HDMI1_TX2_P)
- new net HDMI1_HOTPLUG: Module1.143 (HDMI1_HOTPLUG)
- new net HDMI1_SCL: Module1.147 (HDMI1_SCL)
- new net HDMI1_SDA: Module1.145 (HDMI1_SDA)
- new net ID_SC: Module1.35 (ID_SC)
- new net ID_SD: Module1.36 (ID_SD)
- new net PCIE_CLK_N: Module1.112 (PCIe_CLK_N)
- new net PCIE_CLK_P: Module1.110 (PCIe_CLK_P)
- new net PCIE_CLK_nREQ: Module1.102 (PCIe_CLK_nREQ)
- new net PCIE_RX_N: Module1.118 (PCIe_RX_N)
- new net PCIE_RX_P: Module1.116 (PCIe_RX_P)
- new net PCIE_TX_N: Module1.124 (PCIe_TX_N)
- new net PCIE_TX_P: Module1.122 (PCIe_TX_P)
- new net PCIE_nRST: Module1.109 (PCIe_nRST)
- new net RUN_PG: Module1.92 (RUN_PG)
- new net Reserved: Module1.76 (Reserved)
- new net SD_CLK: Module1.57 (SD_CLK)
- new net SD_CMD: Module1.62 (SD_CMD)
- new net SD_DAT0: Module1.63 (SD_DAT0)
- new net SD_DAT1: Module1.67 (SD_DAT1)
- new net SD_DAT2: Module1.69 (SD_DAT2)
- new net SD_DAT3: Module1.61 (SD_DAT3)
- new net SD_PWR_ON: Module1.75 (SD_PWR_ON)
- new net SYNC_IN: Module1.16 (Ethernet_SYNC_IN(1.8v))
- new net SYNC_OUT: Module1.18 (Ethernet_SYNC_OUT(1.8v))
- new net TRD0_N: Module1.10 (Ethernet_Pair0_N)
- new net TRD0_P: Module1.12 (Ethernet_Pair0_P)
- new net TRD1_N: Module1.6 (Ethernet_Pair1_N)
- new net TRD1_P: Module1.4 (Ethernet_Pair1_P)
- new net TRD2_N: Module1.9 (Ethernet_Pair2_N)
- new net TRD2_P: Module1.11 (Ethernet_Pair2_P)
- new net TRD3_N: Module1.5 (Ethernet_Pair3_N)
- new net TRD3_P: Module1.3 (Ethernet_Pair3_P)
- new net TV_OUT: Module1.111 (VDAC_COMP)
- new net USB2_N: Module1.103 (USB2_N)
- new net USB2_P: Module1.105 (USB2_P)
- new net USBOTG_ID: Module1.101 (USB_OTG_ID)
- new net WL_nDis: J3.1 (Pin_1), Module1.89 (WiFi_nDisable)
- new net nEXTRST: Module1.100 (nEXTRST)
- new net nPWR_LED: Module1.95 (nPI_LED_PWR)
- new net nRPIBOOT: Module1.93 (nRPIBOOT)
- no-connect marks 97 -> 102
Other:
- removed sheet POWER
- note added: "Activity LED"
- note added: "Novatel OEM7xx GNSS receiver"

Commit message: OBC: initialize schematic, spacecraft bus
Parts:
- removed R2: 10k, Resistor_SMD:R_0603_1608Metric, symbol Device:R_Small_US
- removed U2: LTC2854HDD-PBF, LTC2584:DFN-10_DD_LIT, symbol 2024-11-27_15-49-54:LTC2854HDD-PBF
- added U1: ~, symbol HEDGE2:NOVATEL OEM719
- added U2, U8: TCAN1051VDRBRQ1, DRB8_TEX, symbol TCAN1051V:TCAN1051VDRBRQ1
Connections:
- net +3.3v is gone; now on net +3V3: D2.2 (A), Module1.84 (+3.3v_(Output)), Module1.86 (+3.3v_(Output))
- net +5v is gone; now on net +5V: Module1.77 (+5v_(Input)), Module1.79 (+5v_(Input)), Module1.81 (+5v_(Input)), Module1.83 (+5v_(Input)), Module1.85 (+5v_(Input)), Module1.87 (+5v_(Input))
- net BUS5V is gone; now on net 5V_PERM: H2.25, H2.26
- net GND: now also H1.29, H1.30, H1.31, H1.32, H2.29, H2.30, H2.31, H2.32; no longer H2.21, H2.22, H2.23, H2.24
- net ENA_PWR_5: now reaches H2.33
- net PWR_5: now reaches H2.34
- net ENA_PWR_6: now reaches H2.35
- net PWR_6: now reaches H2.36
- net ENA_PWR_7: now reaches H2.37
- net PWR_7: now reaches H2.38
- net ENA_PWR_8: now reaches H2.39
- net PWR_8: now reaches H2.40
- net CHARGE: now reaches H2.43
- net CHARGE: now also H2.44
- net BATT: now reaches H2.45
- net BATT: now also H2.46
- net RBF_A: now reaches H2.47
- net DS_A: now reaches H2.48
- net RBF_B: now reaches H2.49
- net DS_B: now reaches H2.50
- net RBF_C: now reaches H2.51
- net DS_C: now reaches H2.52
- net CAN_A_L: now reaches H1.1
- net CAN_A_L: now also U2.6 (CANL)
- net UART_C_TX: now reaches H1.13
- net UART_C_RX: now reaches H1.15
- net CAN_B_L: now reaches H1.2
- net CAN_B_L: now also U8.6 (CANL)
- net UART_D_TX: now reaches H1.22
- net UART_D_RX: now reaches H1.24
- net 5V_PERM: now reaches H1.25
- net 5V_PERM: now also H1.26
- net CAN_A_H: now reaches H1.3
- net CAN_A_H: now also U2.7 (CANH)
- net UART_E_TX: now reaches H1.38
- net CAN_B_H: now reaches H1.4
- net CAN_B_H: now also U8.7 (CANH)
- net UART_E_RX: now reaches H1.40
- net UART_F_TX: now reaches H1.42
- net UART_F_RX: now reaches H1.44
- net ENA_PWR_1: now reaches H1.45
- net PWR_1: now reaches H1.46
- net ENA_PWR_2: now reaches H1.47
- net PWR_2: now reaches H1.48
- net ENA_PWR_3: now reaches H1.49
- net UART_A_TX: now reaches H1.5
- net PWR_3: now reaches H1.50
- net ENA_PWR_4: now reaches H1.51
- net PWR_4: now reaches H1.52
- net UART_B_TX: now reaches H1.6
- net UART_A_RX: now reaches H1.7
- net UART_B_RX: now reaches H1.8
- net BUS3V3: no longer names the net of H2.27
- net BUS3V3: no longer H2.28
- net Pay1 A: no longer names the net of H1.18
- net Pay1 B: no longer names the net of H1.20
- no-connect marks 102 -> 127
Other:
- note removed: "Novatel OEM7xx GNSS receiver"
- moved on the sheet: H1, H2

Commit message: OBC: schematic input
Parts:
- removed U2, U8: TCAN1051VDRBRQ1, DRB8_TEX, symbol TCAN1051V:TCAN1051VDRBRQ1
- added AE1: Antenna, symbol Device:Antenna
- added J1: AudioJack3, symbol Connector_Audio:AudioJack3
Connections:
- net PWR_1 is gone; now on net +5V: H1.46
- net +5V: no longer Module1.77 (+5v_(Input)), Module1.79 (+5v_(Input)), Module1.81 (+5v_(Input)), Module1.83 (+5v_(Input)), Module1.85 (+5v_(Input)), Module1.87 (+5v_(Input))
- net GND: now also U1.10 (GND), U1.13 (GND), U1.16 (GND), U1.18 (GND), J1.S
- net at U1.11 (TXD1): now also J1.R
- net at U1.12 (RXD1): now also J1.T
- net GNSS_TXD: now reaches U1.14 (TXD2)
- net GNSS_RXD: now reaches U1.15 (RXD2)
- net GNSS_PV: now reaches U1.17 (PV)
- net GNSS_PPS: now reaches U1.19 (PPS)
- net +3V3_OEM719: now reaches U1.2 (3V3)
- net GNSS_NRESET_IN: now reaches U1.5 (nRESET_IN)
- net CAM_GPIO: no longer names the net of Module1.97 (Camera_GPIO)
- net PCIE_CLK_N: no longer names the net of Module1.112 (PCIe_CLK_N)
- net PCIE_CLK_P: no longer names the net of Module1.110 (PCIe_CLK_P)
- net PCIE_CLK_nREQ: no longer names the net of Module1.102 (PCIe_CLK_nREQ)
- net PCIE_RX_N: no longer names the net of Module1.118 (PCIe_RX_N)
- net PCIE_RX_P: no longer names the net of Module1.116 (PCIe_RX_P)
- net PCIE_TX_N: no longer names the net of Module1.124 (PCIe_TX_N)
- net PCIE_TX_P: no longer names the net of Module1.122 (PCIe_TX_P)
- net PCIE_nRST: no longer names the net of Module1.109 (PCIe_nRST)
- net TV_OUT: no longer names the net of Module1.111 (VDAC_COMP)
- net USB2_N: no longer names the net of Module1.103 (USB2_N)
- net USB2_P: no longer names the net of Module1.105 (USB2_P)
- net USBOTG_ID: no longer names the net of Module1.101 (USB_OTG_ID)
- net nEXTRST: no longer names the net of Module1.100 (nEXTRST)
- new net +5V_RPI: Module1.77 (+5v_(Input)), Module1.79 (+5v_(Input)), Module1.81 (+5v_(Input)), Module1.83 (+5v_(Input)), Module1.85 (+5v_(Input)), Module1.87 (+5v_(Input))
- no-connect marks 127 -> 136
Other:
- added sheet INA260_OEM719 (INA260.kicad_sch)
- added sheet INA260_RPI (INA260.kicad_sch)
- added sheet TCAN1051V_A (TCAN1051V.kicad_sch)
- added sheet TCAN1051V_B (TCAN1051V.kicad_sch)
- added sheet TPS543320 (TPS543320.kicad_sch)
- note added: "CONFIG"
- moved on the sheet: U1

Commit message: OBC: initial schematic entry complete
Parts:
- removed R4: 4k7, Resistor_SMD:R_0603_1608Metric, symbol Device:R_Small_US
- added R2: 4k7, Resistor_SMD:R_0805_2012Metric, symbol Device:R_Small_US
- R1: footprint Resistor_SMD:R_0402_1005Metric -> Resistor_SMD:R_0805_2012Metric
- R3: footprint Resistor_SMD:R_0603_1608Metric -> Resistor_SMD:R_0805_2012Metric
- renumbered D2 to D1, J3 to J2, TP3 to TP1
Connections:
- net GPIO14 is gone; now on net CAN_A_TXD: Module1.55 (GPIO14)
- net GPIO15 is gone; now on net CAN_A_RXD: Module1.51 (GPIO15)
- net GPIO16 is gone; now on net CAN_A_S: Module1.29 (GPIO16)
- net GPIO2 is gone; now on net CAN_B_S: Module1.58 (GPIO2)
- net GPIO4 is gone; now on net GNSS_TXD: Module1.54 (GPIO4)
- net GPIO5 is gone; now on net GNSS_RXD: Module1.34 (GPIO5)
- net ID_SC is gone; now on net CAN_B_RXD: Module1.35 (ID_SC)
- net ID_SD is gone; now on net CAN_B_TXD: Module1.36 (ID_SD)
- net UART_D_RX is gone; now on net GPIO9: H1.24
- net UART_D_TX is gone; now on net GPIO8: H1.22
- net UART_E_RX is gone; now on net GPIO13: H1.40
- net UART_E_TX is gone; now on net GPIO12: H1.38
- net +3V3: now also R2.2
- net +5V: no longer H1.46
- net SCL0: now also R2.1; no longer R3.1
- net SDA0: now also R3.1
- net +3V3_OEM719 renamed TPS543320/VOUT
- net +5V_RPI renamed +5V_CM4
- net PWR_2 renamed +5V_GNSS
- net nRPIBOOT renamed nCM4BOOT
- new net +5V_MPU: H1.46
Other:
- sheet INA260_RPI renamed INA260_CM4
- note added: "0x40"
- note added: "0x41"
- note added: "SPACECRAFT BUS MAPPINGS"
- note added: "UART4"
- note added: "UART5"
- moved on the sheet: AE1, J1, MH1, MH2, MH3, MH4, U1

Commit message: OBC: preliminary layout
Parts:
- removed J1: AudioJack3, symbol Connector_Audio:AudioJack3
- removed R1: 1k, Resistor_SMD:R_0805_2012Metric, symbol Device:R
- removed TP1: TestPoint, TestPoint:TestPoint_Pad_2.0x2.0mm, symbol Connector:TestPoint
- added C1, C2: 0u1, Capacitor_SMD:C_0805_2012Metric, symbol Device:C_Small
- added D2: LED GREEN, LED_SMD:LED_0805_2012Metric, symbol Device:LED
- added J1: 54-00175, 54_00175-audio-jack:TENSILITY_54-00175, symbol 54-00175-audio-jack:54-00175
- added JP1, JP2, JP3, JP4: ~, Jumper:SolderJumper-2_P1.3mm_Open_RoundedPad1.0x1.5mm, symbol Jumper:SolderJumper_2_Open
- added R1, R2, R3, R4: 60, Resistor_SMD:R_0805_2012Metric, symbol Device:R_Small_US
- added R5, R6: 1k, Resistor_SMD:R_0805_2012Metric, symbol Device:R_Small_US
- added U1, U8: 74LVC1GU04DBV, Package_TO_SOT_SMD:SOT-23-5, symbol 74xGxx:74LVC1GU04
- AE1: footprint (none) -> Connector_Coaxial:SMA_Amphenol_901-144_Vertical
- D1: value LED Green -> LED RED; footprint LED_SMD:LED_0603_1608Metric -> LED_SMD:LED_0805_2012Metric; Field4 Digikey -> (none); Field5 LTST-S270KGKT -> (none); Field6 SML-A12M8TT86N -> (none); Field7 Rohm -> (none); Field8 650263301 -> (none); Part Description Green 572nm LED Indication - Discrete 2.2V 2-SMD, No Lead -> (none)
- H1, H2: Arrow Part Number (none) -> ESQ-126-39-G-D
- J2: footprint Connector_PinHeader_2.54mm:PinHeader_1x03_P2.54mm_Vertical -> Connector_PinSocket_2.00mm:PinSocket_2x10_P2.00mm_Vertical
- MH1, MH2, MH3, MH4: footprint MountingHole-VST104:MountingHole_3.2mm_M3_Pad_Via -> MountingHole:MountingHole_3.2mm_M3_Pad_Via
- Module1: footprint CM4IO:Raspberry-Pi-4-Compute-Module -> CM4102008:MODULE_CM4102008
- U2: renamed from U1; value ~ -> OEM719; footprint (none) -> Novatel:OEM719
- renumbered R2 to R7, R3 to R8
Connections:
- net GPIO_VREF is gone; now on net +3V3: Module1.78 (GPIO_VREF(1.8v/3.3v_Input))
- net +3V3: now also D2.2 (A), U1.5 (VCC), U8.5 (VCC)
- net +5V_CM4: no longer Module1.79 (+5v_(Input)), Module1.81 (+5v_(Input)), Module1.83 (+5v_(Input)), Module1.85 (+5v_(Input))
- net CAN_A_H: now also JP1.2 (B), JP3.2 (B)
- net CAN_A_L: now also JP2.1 (A), JP4.1 (A)
- net GND: now also C1.2, C2.2, J1.1, U1.3 (GND), U8.3 (GND)
- net nPWR_LED: now also U1.2
- net at D1.1 (K): now also R5.2
- net PI_nLED_Activity: now reaches Module1.21 (PI_nLED_Activity)
- net PI_nLED_Activity: now also U8.2
- net at U2.11 (TXD1): now also J1.3
- net at U2.12 (RXD1): now also J1.2
- new net: C2.1, R3.2, R4.1
- new net: R5.1, U1.4
- new net: JP2.2 (B), R2.2
- new net: R6.1, U8.4
- new net: JP1.1 (A), R1.1
- new net: C1.1, R1.2, R2.1
- new net: D2.1 (K), R6.2
- new net: JP4.2 (B), R4.2
- new net: JP3.1 (A), R3.1
- no-connect marks 136 -> 138
Other:
- note added: "GNSS CONFIG"
- note added: "PWR LED"
- note removed: "Activity LED"
- note removed: "CONFIG"

Commit message: OBC: start PCB layout
Parts:
- removed J2: Conn_01x03, Connector_PinSocket_2.00mm:PinSocket_2x10_P2.00mm_Vertical, symbol Connector_Generic:Conn_01x03
- removed U1, U8: 74LVC1GU04DBV, Package_TO_SOT_SMD:SOT-23-5, symbol 74xGxx:74LVC1GU04
- added JP5: WiFi_nDisable, Jumper:SolderJumper-2_P1.3mm_Open_RoundedPad1.0x1.5mm, symbol Jumper:Jumper_2_Bridged
- added JP6: BT_nDisable, Jumper:SolderJumper-2_P1.3mm_Bridged_RoundedPad1.0x1.5mm, symbol Jumper:Jumper_2_Bridged
- R5: renamed from R6; value 1k -> 39
- R6: renamed from R5; value 1k -> 45
- renumbered D2 to D1, D1 to D2, U2 to U1
Connections:
- net GPIO11 is gone; now on net GNSS_NRESET_IN: Module1.38 (GPIO11)
- net GPIO17 is gone; now on net GNSS_PV: Module1.50 (GPIO17)
- net GPIO22 is gone; now on net GNSS_PPS: Module1.46 (GPIO22)
- net +3V3: no longer D1.2 (A), D2.2 (A)
- net +5V_CM4: now also Module1.79 (+5v_(Input)), Module1.81 (+5v_(Input)), Module1.83 (+5v_(Input)), Module1.85 (+5v_(Input))
- net CAN_A_H: no longer JP3.2 (B)
- net CAN_A_L: no longer JP4.1 (A)
- net CAN_B_H: now also JP3.2 (B)
- net CAN_B_L: now also JP4.1 (A)
- net GND: now also D1.1 (K), D2.1 (K), JP5.1 (A), JP6.2 (B)
- net PI_nLED_Activity: now also R5.1
- net nPWR_LED: now also R6.1
- net at AE1.1 (A): now also U1.21 (ANT)
- net at R6.2: now also D2.2 (A); no longer D2.1 (K)
- net at R5.2: now also D1.2 (A); no longer D1.1 (K)
- net +1.8v: no longer names the net of Module1.88 (+1.8v_(Output)), Module1.90 (+1.8v_(Output))
- net AIN0: no longer names the net of Module1.96 (AnalogIP1)
- net AIN1: no longer names the net of Module1.94 (AnalogIP0)
- net BT_nDis: no longer names the net of Module1.91 (BT_nDisable)
- net BT_nDis: now also JP6.1 (A)
- net CAM0_C_N: no longer names the net of Module1.140 (CAM0_C_N)
- net CAM0_C_P: no longer names the net of Module1.142 (CAM0_C_P)
- net CAM0_D0_N: no longer names the net of Module1.128 (CAM0_D0_N)
- net CAM0_D0_P: no longer names the net of Module1.130 (CAM0_D0_P)
- net CAM0_D1_N: no longer names the net of Module1.134 (CAM0_D1_N)
- net CAM0_D1_P: no longer names the net of Module1.136 (CAM0_D1_P)
- net CAM1_C_N: no longer names the net of Module1.127 (CAM1_C_N)
- net CAM1_C_P: no longer names the net of Module1.129 (CAM1_C_P)
- net CAM1_D0_N: no longer names the net of Module1.115 (CAM1_D0_N)
- net CAM1_D0_P: no longer names the net of Module1.117 (CAM1_D0_P)
- net CAM1_D1_N: no longer names the net of Module1.121 (CAM1_D1_N)
- net CAM1_D1_P: no longer names the net of Module1.123 (CAM1_D1_P)
- net CAM1_D2_N: no longer names the net of Module1.133 (CAM1_D2_N)
- net CAM1_D2_P: no longer names the net of Module1.135 (CAM1_D2_P)
- net CAM1_D3_N: no longer names the net of Module1.139 (CAM1_D3_N)
- net CAM1_D3_P: no longer names the net of Module1.141 (CAM1_D3_P)
- net DSI0_C_N: no longer names the net of Module1.169 (DSI0_C_N)
- net DSI0_C_P: no longer names the net of Module1.171 (DSI0_C_P)
- net DSI0_D0_N: no longer names the net of Module1.157 (DSI0_D0_N)
- net DSI0_D0_P: no longer names the net of Module1.159 (DSI0_D0_P)
- net DSI0_D1_N: no longer names the net of Module1.163 (DSI0_D1_N)
- net DSI0_D1_P: no longer names the net of Module1.165 (DSI0_D1_P)
- net DSI1_C_N: no longer names the net of Module1.187 (DSI1_C_N)
- net DSI1_C_P: no longer names the net of Module1.189 (DSI1_C_P)
- net DSI1_D0_N: no longer names the net of Module1.175 (DSI1_D0_N)
- net DSI1_D0_P: no longer names the net of Module1.177 (DSI1_D0_P)
- net DSI1_D1_N: no longer names the net of Module1.181 (DSI1_D1_N)
- net DSI1_D1_P: no longer names the net of Module1.183 (DSI1_D1_P)
- net DSI1_D2_N: no longer names the net of Module1.193 (DSI1_D2_N)
- net DSI1_D2_P: no longer names the net of Module1.195 (DSI1_D2_P)
- net DSI1_D3_N: no longer names the net of Module1.194 (DSI1_D3_N)
- net DSI1_D3_P: no longer names the net of Module1.196 (DSI1_D3_P)
- net EEPROM_nWP: no longer names the net of Module1.20 (EEPROM_nWP)
- net ETH_LEDG: no longer names the net of Module1.17 (Ethernet_nLED2(3.3v))
- net ETH_LEDY: no longer names the net of Module1.15 (Ethernet_nLED3(3.3v))
- net GLOBAL_EN: no longer names the net of Module1.99 (Global_EN)
- net GPIO10: no longer names the net of Module1.44 (GPIO10)
- net GPIO12 renamed UART_DATA_TX
- net GPIO13 renamed UART_DATA_RX
- net GPIO18: no longer names the net of Module1.49 (GPIO18)
- net GPIO19: no longer names the net of Module1.26 (GPIO19)
- net GPIO20: no longer names the net of Module1.27 (GPIO20)
- net GPIO21: no longer names the net of Module1.25 (GPIO21)
- net GPIO23: no longer names the net of Module1.47 (GPIO23)
- net GPIO24: no longer names the net of Module1.45 (GPIO24)
- net GPIO25: no longer names the net of Module1.41 (GPIO25)
- net GPIO26: no longer names the net of Module1.24 (GPIO26)
- net GPIO27: no longer names the net of Module1.48 (GPIO27)
- net GPIO3: no longer names the net of Module1.56 (GPIO3)
- net GPIO6: no longer names the net of Module1.30 (GPIO6)
- net GPIO7: no longer names the net of Module1.37 (GPIO7)
- net GPIO8 renamed UART_COMM_TX
- net GPIO9 renamed UART_COMM_RX
- net HDMI0_CEC: no longer names the net of Module1.151 (HDMI0_CEC)
- net HDMI0_CK_N: no longer names the net of Module1.190 (HDMI0_CLK_N)
- net HDMI0_CK_P: no longer names the net of Module1.188 (HDMI0_CLK_P)
- net HDMI0_D0_N: no longer names the net of Module1.184 (HDMI0_TX0_N)
- net HDMI0_D0_P: no longer names the net of Module1.182 (HDMI0_TX0_P)
- net HDMI0_D1_N: no longer names the net of Module1.178 (HDMI0_TX1_N)
- net HDMI0_D1_P: no longer names the net of Module1.176 (HDMI0_TX1_P)
- net HDMI0_D2_N: no longer names the net of Module1.172 (HDMI0_TX2_N)
- net HDMI0_D2_P: no longer names the net of Module1.170 (HDMI0_TX2_P)
- net HDMI0_HOTPLUG: no longer names the net of Module1.153 (HDMI0_HOTPLUG)
- net HDMI0_SCL: no longer names the net of Module1.200 (HDMI0_SCL)
- net HDMI0_SDA: no longer names the net of Module1.199 (HDMI0_SDA)
- net HDMI1_CEC: no longer names the net of Module1.149 (HDMI1_CEC)
- net HDMI1_CK_N: no longer names the net of Module1.166 (HDMI1_CLK_N)
- net HDMI1_CK_P: no longer names the net of Module1.164 (HDMI1_CLK_P)
- net HDMI1_D0_N: no longer names the net of Module1.160 (HDMI1_TX0_N)
- net HDMI1_D0_P: no longer names the net of Module1.158 (HDMI1_TX0_P)
- net HDMI1_D1_N: no longer names the net of Module1.154 (HDMI1_TX1_N)
- net HDMI1_D1_P: no longer names the net of Module1.152 (HDMI1_TX1_P)
- net HDMI1_D2_N: no longer names the net of Module1.148 (HDMI1_TX2_N)
- net HDMI1_D2_P: no longer names the net of Module1.146 (HDMI1_TX2_P)
- net HDMI1_HOTPLUG: no longer names the net of Module1.143 (HDMI1_HOTPLUG)
- net HDMI1_SCL: no longer names the net of Module1.147 (HDMI1_SCL)
- net HDMI1_SDA: no longer names the net of Module1.145 (HDMI1_SDA)
- net RUN_PG: no longer names the net of Module1.92 (RUN_PG)
- net Reserved: no longer names the net of Module1.76 (Reserved)
- net SD_CLK: no longer names the net of Module1.57 (SD_CLK)
- net SD_CMD: no longer names the net of Module1.62 (SD_CMD)
- net SD_DAT0: no longer names the net of Module1.63 (SD_DAT0)
- net SD_DAT1: no longer names the net of Module1.67 (SD_DAT1)
- net SD_DAT2: no longer names the net of Module1.69 (SD_DAT2)
- net SD_DAT3: no longer names the net of Module1.61 (SD_DAT3)
- net SD_PWR_ON: no longer names the net of Module1.75 (SD_PWR_ON)
- net SYNC_IN: no longer names the net of Module1.16 (Ethernet_SYNC_IN(1.8v))
- net SYNC_OUT: no longer names the net of Module1.18 (Ethernet_SYNC_OUT(1.8v))
- net TRD0_N: no longer names the net of Module1.10 (Ethernet_Pair0_N)
- net TRD0_P: no longer names the net of Module1.12 (Ethernet_Pair0_P)
- net TRD1_N: no longer names the net of Module1.6 (Ethernet_Pair1_N)
- net TRD1_P: no longer names the net of Module1.4 (Ethernet_Pair1_P)
- net TRD2_N: no longer names the net of Module1.9 (Ethernet_Pair2_N)
- net TRD2_P: no longer names the net of Module1.11 (Ethernet_Pair2_P)
- net TRD3_N: no longer names the net of Module1.5 (Ethernet_Pair3_N)
- net TRD3_P: no longer names the net of Module1.3 (Ethernet_Pair3_P)
- net WL_nDis: no longer names the net of Module1.89 (WiFi_nDisable)
- net WL_nDis: now also JP5.2 (B)
- net nCM4BOOT: no longer names the net of Module1.93 (nRPIBOOT)
- no-connect marks 138 -> 204
Other:
- note added: "ACTIVITY LED"
- moved on the sheet: AE1, D1, D2, R5, R6
