File: COMM.kicad_sch (KiCad schematic)
At the start: 42 parts, among them J10 Conn_01x03, J6 BOOTSEL, J7 731000115, J8 SS4-10-3.50-X-D-K-TR, J9 10118194-0001LF, U3 LTC2854HDD-PBF, U3 SN74LVC1T45DBVR, U4 RFM69HCW 900MHz, U4 W25Q16JVUXIQ TR, U5 DMG2305UX-13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

Commit message: OBC: initial schematic entry complete
Parts:
- removed C10: 10p, Capacitor_SMD:C_0603_1608Metric, symbol Device:C_Small
- removed C11, C3, C4: 47u, Capacitor_SMD:C_0603_1608Metric, symbol Device:C_Small
- removed C3: 100n, Capacitor_SMD:C_0603_1608Metric, symbol Device:C_Small
- removed C4: 2u2, Capacitor_SMD:C_0603_1608Metric, symbol Device:C_Small
- removed C5, C6: 15p, Capacitor_SMD:C_0603_1608Metric, symbol Device:C_Small
- removed C7: 22p, Capacitor_SMD:C_0603_1608Metric, symbol Device:C_Small
- removed C8: 5p, Capacitor_SMD:C_0603_1608Metric, symbol Device:C_Small
- removed C9: 4u7, Capacitor_SMD:C_0603_1608Metric, symbol Device:C_Small
- removed CR1: MBR120VLSFT1G, MBR120VLS:SDO_SOD-123FL_ONS, symbol 2024-12-09_13-52-28:MBR120VLSFT1G
- removed E1: YCIS003AA, YCIS003AA:XDCR_YCIS003AA, symbol YCIS003AA:YCIS003AA
- removed H3, H4: Conn_02x26_Odd_Even, ESQ-126-39-G-D:ESQ-126-Y-X-D, symbol ESQ-126-39-G-D:ESQ-126-39-G-D
- removed J10: Conn_01x03, Connector_PinHeader_2.54mm:PinHeader_1x03_P2.54mm_Horizontal, symbol Connector_Generic:Conn_01x03
- removed J6: BOOTSEL, Connector_PinHeader_2.54mm:PinHeader_1x02_P2.54mm_Horizontal, symbol Connector_Generic:Conn_01x02
- removed J7: 731000115, 731000115_SMA:COAX4GND_731000115_MOL, symbol 2024-12-06_19-24-29:731000115
- removed J8: SS4-10-3.50-X-D-K-TR, ESQ-126-39-G-D:ESQ-126-Y-X-D, symbol SS4-10-3.50-X-D-K-TR:SS4-10-3.50-X-D-K-TR
- removed J9: 10118194-0001LF, 10118194_0001LF:AMPHENOL_10118194-0001LF, symbol 10118194-0001LF:10118194-0001LF
- removed JP1: Jumper_2_Open, Connector_PinHeader_2.54mm:PinHeader_1x02_P2.54mm_Vertical, symbol Jumper:Jumper_2_Open
- removed R10, R9: 4k7, Resistor_SMD:R_0603_1608Metric, symbol Device:R_Small_US
- removed R5, R6: 1k, Resistor_SMD:R_0603_1608Metric, symbol Device:R_Small_US
- removed R5: 10k, Resistor_SMD:R_0603_1608Metric, symbol Device:R_Small_US
- removed R6: 0, Resistor_SMD:R_0603_1608Metric, symbol Device:R_Small_US
- removed R7, R8: 27, Resistor_SMD:R_0603_1608Metric, symbol Device:R_Small_US
- removed R7, R8: 4u7, Resistor_SMD:R_0603_1608Metric, symbol Device:R_Small_US
- removed U3: LTC2854HDD-PBF, LTC2584:DFN-10_DD_LIT, symbol 2024-11-27_15-49-54:LTC2854HDD-PBF
- removed U3: SN74LVC1T45DBVR, SN74LVC1T45DBVR:SOT95P280X145-6N, symbol SN74LVC1T45DBVR:SN74LVC1T45DBVR
- removed U4: RFM69HCW 900MHz, COM_13909:RFM69HCW_SPK, symbol COM_13909:COM-13909
- removed U4: W25Q16JVUXIQ TR, W25Q16JVUXIQ:USON-8_UX_2x3x0p6_WIN, symbol 2024-12-07_14-34-38:W25Q16JVUXIQ_TR
- removed U5: DMG2305UX-13, DMG2305UX:SOT91P240X110-3N, symbol DMG2305UX-13:DMG2305UX-13
- removed U6: RP2040, RP2040:QFN56_7X7_RPI, symbol MCU_RaspberryPi:RP2040
- removed X1: ABM8-272-T3, ABM8_272_T3:ABM8-272-T3_ABR, symbol 2024-12-07_14-51-31:ABM8-272-T3
Connections:
- no-connect marks 126 -> 0
Other:
- removed sheet POWER
- note removed: "FOR GROUND TESTING ONLY DISABLED BEFORE FLIGHT"

Commit message: OBC: preliminary layout
Parts:
- MH5, MH6, MH7, MH8: footprint MountingHole-VST104:MountingHole_3.2mm_M3_Pad_Via -> MountingHole:MountingHole_3.2mm_M3_Pad_Via
Changed lines of the file:
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@@
 			)
 		)
-		(property "Footprint" "MountingHole-VST104:MountingHole_3.2mm_M3_Pad_Via"
+		(property "Footprint" "MountingHole:MountingHole_3.2mm_M3_Pad_Via"
 			(at 312.42 223.52 0)
 			(effects
@@
 			)
 		)
-		(property "Footprint" "MountingHole-VST104:MountingHole_3.2mm_M3_Pad_Via"
+		(property "Footprint" "MountingHole:MountingHole_3.2mm_M3_Pad_Via"
 			(at 308.61 217.17 0)
 			(effects
@@
 			)
 		)
-		(property "Footprint" "MountingHole-VST104:MountingHole_3.2mm_M3_Pad_Via"
+		(property "Footprint" "MountingHole:MountingHole_3.2mm_M3_Pad_Via"
 			(at 326.39 223.52 0)
 			(effects
@@
 		(dnp no)
 		(fields_autoplaced yes)
-		(property "Reference" "#PWR068"
+		(property "Reference" "#PWR039"
 			(at 320.04 234.95 0)
 			(effects
@@
 			(project "Avionics"
 				(path "/ace5002f-3cbc-4a0a-869b-0e31ebd905b7/617751c8-9e63-43a2-807c-be0203e52cd6"
-					(reference "#PWR068")
+					(reference "#PWR039")
 					(unit 1)
 				)
@@
 			)
 		)
-		(property "Footprint" "MountingHole-VST104:MountingHole_3.2mm_M3_Pad_Via"
+		(property "Footprint" "MountingHole:MountingHole_3.2mm_M3_Pad_Via"
 			(at 321.31 217.17 0)
 			(effects

Commit message: OBC: Continue PCB lauout
Parts:
- added H1COMM1, H2COMM1: Conn_02x26_Odd_Even, ESQ-126-39-G-D:SAMTEC_ESQ-126-39-G-D, symbol ESQ-126-39-G-D:ESQ-126-39-G-D
Connections:
- net GND: now also H1COMM1.29, H1COMM1.30, H1COMM1.31, H1COMM1.32, H2COMM1.29, H2COMM1.30, H2COMM1.31, H2COMM1.32
- new net 5V_PERM: H1COMM1.25, H1COMM1.26, H2COMM1.25, H2COMM1.26
- new net BATT: H2COMM1.45, H2COMM1.46
- new net CAN_A_H: H1COMM1.03
- new net CAN_A_L: H1COMM1.01
- new net CAN_B_H: H1COMM1.04
- new net CAN_B_L: H1COMM1.02
- new net CHARGE: H2COMM1.43, H2COMM1.44
- new net DS_A: H2COMM1.48
- new net DS_B: H2COMM1.50
- new net DS_C: H2COMM1.52
- new net ENA_PWR_1: H1COMM1.45
- new net ENA_PWR_2: H1COMM1.47
- new net ENA_PWR_3: H1COMM1.49
- new net ENA_PWR_4: H1COMM1.51
- new net ENA_PWR_5: H2COMM1.33
- new net ENA_PWR_6: H2COMM1.35
- new net ENA_PWR_7: H2COMM1.37
- new net ENA_PWR_8: H2COMM1.39
- new net PWR_1: H1COMM1.46
- new net PWR_2: H1COMM1.48
- new net PWR_3: H1COMM1.50
- new net PWR_4: H1COMM1.52
- new net PWR_5: H2COMM1.34
- new net PWR_6: H2COMM1.36
- new net PWR_7: H2COMM1.38
- new net PWR_8: H2COMM1.40
- new net RBF_A: H2COMM1.47
- new net RBF_B: H2COMM1.49
- new net RBF_C: H2COMM1.51
- new net UART_A_RX: H1COMM1.07
- new net UART_A_TX: H1COMM1.05
- new net UART_B_RX: H1COMM1.08
- new net UART_B_TX: H1COMM1.06
- new net UART_C_RX: H1COMM1.15
- new net UART_C_TX: H1COMM1.13
- new net UART_D_RX: H1COMM1.24
- new net UART_D_TX: H1COMM1.22
- new net UART_E_RX: H1COMM1.40
- new net UART_E_TX: H1COMM1.38
- new net UART_F_RX: H1COMM1.44
- new net UART_F_TX: H1COMM1.42
- no-connect marks 0 -> 88
