File: EPS.kicad_sch (KiCad schematic)
At the start: 26 parts, among them J11 RBFTEST, J12 G125-MH10805M4-1AD1ADP, J13 Barrel_Jack_Switch_MountingPin, Q1 NVTFS5C454NLTAG, Q2 NVTFS5C454NLTAG, Q3 NVTFS5C454NLTAG, Q4 NVTFS5C454NLTAG, Q5 NVTFS5C454NLTAG, SW3 MC 7792N14 (NO), U7 LTC2854HDD-PBF

Commit message: OBC: initial schematic entry complete
Parts:
- removed BT1: 9.6V 3S 3x26650 LiFePO4, HEDGE:9.6V 3S 3x26650 LiFePO4, symbol Device:Battery_Cell
- removed CR2 (x2), CR3, CR4, CR5: BAS316,115, Diode_SMD:D_SOD-323, symbol BAS716:BAS716_115
- removed H5, H6: Conn_02x26_Odd_Even, ESQ-126-39-G-D:ESQ-126-Y-X-D, symbol ESQ-126-39-G-D:ESQ-126-39-G-D
- removed J11: RBFTEST, Connector_PinHeader_2.54mm:PinHeader_1x02_P2.54mm_Horizontal, symbol Connector_Generic:Conn_01x02
- removed J12: G125-MH10805M4-1AD1ADP, G125-MH10805M4:HARWIN_G125-MH10805M4-1AD1ADP, symbol G125-MH10805M4-1AD1ADP:G125-MH10805M4-1AD1ADP
- removed J13: Barrel_Jack_Switch_MountingPin, Connector_BarrelJack:BarrelJack_Wuerth_694108106102_2.5x5.5mm, symbol Connector:Barrel_Jack_Switch_MountingPin
- removed Q1, Q2, Q3, Q4, Q5: NVTFS5C454NLTAG, NVTFS5C478NLTAG:NVTFS6H854NTAG, symbol NVTFS5C478NLTAG:NVTFS5C478NLTAG
- removed R11: 4u7, Resistor_SMD:R_0603_1608Metric, symbol Device:R_Small_US
- removed R12: 10k, Resistor_SMD:R_0603_1608Metric, symbol Device:R_Small_US
- removed R13, R14: 4k7, Resistor_SMD:R_0603_1608Metric, symbol Device:R_Small_US
- removed SW3: MC 7792N14 (NO), McMasterCarr:7792N14, symbol Switch:SW_SPDT
- removed U7: LTC2854HDD-PBF, LTC2584:DFN-10_DD_LIT, symbol 2024-11-27_15-49-54:LTC2854HDD-PBF
Connections:
- no-connect marks 96 -> 0
Other:
- removed sheet INA260 BATT1
- removed sheet POWER
- removed sheet RP2040
- note removed: "FROM DECK PCB 3.3V LOGIC LEVEL"
- note removed: "GSE-1-N"
- note removed: "GSE-1-P"
- note removed: "HEDGE POWER INHIBIT RBF PIN DISCONNECTS INTERNAL BATTERY GSE1 INHIBIT IS ON THE DECK PCB"
- note removed: "HEDGE-COMM"
- note removed: "HEDGE-DATA"
- note removed: "HEDGE-OBC"
- note removed: "RBF PIN TELLING HEDGE THAT IT IS IN GROUND TESTING MODE, NOT FLIGHT MODE"

Commit message: OBC: preliminary layout
Parts:
- MH10, MH11, MH12, MH9: footprint MountingHole-VST104:MountingHole_3.2mm_M3_Pad_Via -> MountingHole:MountingHole_3.2mm_M3_Pad_Via
Changed lines of the file:
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@@
 			)
 		)
-		(property "Footprint" "MountingHole-VST104:MountingHole_3.2mm_M3_Pad_Via"
+		(property "Footprint" "MountingHole:MountingHole_3.2mm_M3_Pad_Via"
 			(at 322.58 215.9 0)
 			(effects
@@
 			)
 		)
-		(property "Footprint" "MountingHole-VST104:MountingHole_3.2mm_M3_Pad_Via"
+		(property "Footprint" "MountingHole:MountingHole_3.2mm_M3_Pad_Via"
 			(at 309.88 215.9 0)
 			(effects
@@
 		(dnp no)
 		(fields_autoplaced yes)
-		(property "Reference" "#PWR080"
+		(property "Reference" "#PWR040"
 			(at 321.31 233.68 0)
 			(effects
@@
 			(project "Avionics"
 				(path "/ace5002f-3cbc-4a0a-869b-0e31ebd905b7/662a4538-a857-4d47-9892-e46e278fb04f"
-					(reference "#PWR080")
+					(reference "#PWR040")
 					(unit 1)
 				)
@@
 			)
 		)
-		(property "Footprint" "MountingHole-VST104:MountingHole_3.2mm_M3_Pad_Via"
+		(property "Footprint" "MountingHole:MountingHole_3.2mm_M3_Pad_Via"
 			(at 327.66 222.25 0)
 			(effects
@@
 			)
 		)
-		(property "Footprint" "MountingHole-VST104:MountingHole_3.2mm_M3_Pad_Via"
+		(property "Footprint" "MountingHole:MountingHole_3.2mm_M3_Pad_Via"
 			(at 313.69 222.25 0)
 			(effects

Commit message: OBC: Continue PCB lauout
Parts:
- added H1EPS1, H2EPS1: Conn_02x26_Odd_Even, ESQ-126-39-G-D:SAMTEC_ESQ-126-39-G-D, symbol ESQ-126-39-G-D:ESQ-126-39-G-D
Connections:
- net GND: now also H1EPS1.29, H1EPS1.30, H1EPS1.31, H1EPS1.32, H2EPS1.29, H2EPS1.30, H2EPS1.31, H2EPS1.32
- new net 5V_PERM: H1EPS1.25, H1EPS1.26, H2EPS1.25, H2EPS1.26
- new net BATT: H2EPS1.45, H2EPS1.46
- new net CAN_A_H: H1EPS1.03
- new net CAN_A_L: H1EPS1.01
- new net CAN_B_H: H1EPS1.04
- new net CAN_B_L: H1EPS1.02
- new net CHARGE: H2EPS1.43, H2EPS1.44
- new net DS_A: H2EPS1.48
- new net DS_B: H2EPS1.50
- new net DS_C: H2EPS1.52
- new net ENA_PWR_1: H1EPS1.45
- new net ENA_PWR_2: H1EPS1.47
- new net ENA_PWR_3: H1EPS1.49
- new net ENA_PWR_4: H1EPS1.51
- new net ENA_PWR_5: H2EPS1.33
- new net ENA_PWR_6: H2EPS1.35
- new net ENA_PWR_7: H2EPS1.37
- new net ENA_PWR_8: H2EPS1.39
- new net PWR_1: H1EPS1.46
- new net PWR_2: H1EPS1.48
- new net PWR_3: H1EPS1.50
- new net PWR_4: H1EPS1.52
- new net PWR_5: H2EPS1.34
- new net PWR_6: H2EPS1.36
- new net PWR_7: H2EPS1.38
- new net PWR_8: H2EPS1.40
- new net RBF_A: H2EPS1.47
- new net RBF_B: H2EPS1.49
- new net RBF_C: H2EPS1.51
- new net UART_A_RX: H1EPS1.07
- new net UART_A_TX: H1EPS1.05
- new net UART_B_RX: H1EPS1.08
- new net UART_B_TX: H1EPS1.06
- new net UART_C_RX: H1EPS1.15
- new net UART_C_TX: H1EPS1.13
- new net UART_D_RX: H1EPS1.24
- new net UART_D_TX: H1EPS1.22
- new net UART_E_RX: H1EPS1.40
- new net UART_E_TX: H1EPS1.38
- new net UART_F_RX: H1EPS1.44
- new net UART_F_TX: H1EPS1.42
- no-connect marks 0 -> 88
