File: INA260.kicad_sch (KiCad schematic)
At the start: 0 parts

Commit message: OBC: schematic input
Parts:
- added C21: 0.1u, Capacitor_SMD:C_0603_1608Metric, symbol Device:C_Small
- added U10: INA260AIPWR, INA260AIPWR:PW0016A_L, symbol 2024-11-27_17-29-01:INA260AIPWR
Connections:
- new net A0: U10.5 (A0)
- new net A1: U10.4 (A1)
- new net GND: C21.1, U10.11 (GND), U10.6 (GND)
- new net LOAD: U10.14 (IN-), U10.15 (IN-), U10.16 (IN-)
- new net SCL: U10.9 (SCL)
- new net SDA: U10.8 (SDA)
- new net SOURCE: U10.1 (IN+), U10.12 (VBUS), U10.2 (IN+), U10.3 (IN+)
- new net VS: C21.2, U10.10 (VS)
- no-connect marks 0 -> 2

Commit message: OBC: initial schematic entry complete
Parts:
- C17: renamed from C21; footprint Capacitor_SMD:C_0603_1608Metric -> Capacitor_SMD:C_0805_2012Metric
Changed lines of the file:
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@@
 		(dnp no)
 		(fields_autoplaced yes)
-		(property "Reference" "C21"
+		(property "Reference" "C17"
 			(at 176.53 106.6864 90)
 			(effects
@@
 			)
 		)
-		(property "Footprint" "Capacitor_SMD:C_0603_1608Metric"
+		(property "Footprint" "Capacitor_SMD:C_0805_2012Metric"
 			(at 182.88 106.68 0)
 			(effects
@@
 			(project "Avionics"
 				(path "/ace5002f-3cbc-4a0a-869b-0e31ebd905b7/893aef5a-59ff-410b-9a71-9930aaf04e9f/740c0668-bfac-47e0-b7b8-de442260ca55"
-					(reference "C21")
+					(reference "C17")
 					(unit 1)
 				)
 				(path "/ace5002f-3cbc-4a0a-869b-0e31ebd905b7/893aef5a-59ff-410b-9a71-9930aaf04e9f/9fa6cc5e-a76a-4d58-8af7-47af14171882"
-					(reference "C20")
+					(reference "C24")
 					(unit 1)
 				)
@@
 		(dnp no)
 		(fields_autoplaced yes)
-		(property "Reference" "#PWR071"
+		(property "Reference" "#PWR091"
 			(at 231.14 152.4 0)
 			(effects
@@
 			(project "Avionics"
 				(path "/ace5002f-3cbc-4a0a-869b-0e31ebd905b7/893aef5a-59ff-410b-9a71-9930aaf04e9f/740c0668-bfac-47e0-b7b8-de442260ca55"
-					(reference "#PWR071")
+					(reference "#PWR091")
 					(unit 1)
 				)
 				(path "/ace5002f-3cbc-4a0a-869b-0e31ebd905b7/893aef5a-59ff-410b-9a71-9930aaf04e9f/9fa6cc5e-a76a-4d58-8af7-47af14171882"
-					(reference "#PWR011")
+					(reference "#PWR0100")
 					(unit 1)
 				)
@@
 				)
 				(path "/ace5002f-3cbc-4a0a-869b-0e31ebd905b7/893aef5a-59ff-410b-9a71-9930aaf04e9f/9fa6cc5e-a76a-4d58-8af7-47af14171882"
-					(reference "U9")
+					(reference "U13")
 					(unit 1)
 				)
@@
 		(dnp no)
 		(fields_autoplaced yes)
-		(property "Reference" "#PWR070"
+		(property "Reference" "#PWR090"
 			(at 182.88 93.98 0)
 			(effects
@@
 			(project "Avionics"
 				(path "/ace5002f-3cbc-4a0a-869b-0e31ebd905b7/893aef5a-59ff-410b-9a71-9930aaf04e9f/740c0668-bfac-47e0-b7b8-de442260ca55"
-					(reference "#PWR070")
+					(reference "#PWR090")
 					(unit 1)
 				)
 				(path "/ace5002f-3cbc-4a0a-869b-0e31ebd905b7/893aef5a-59ff-410b-9a71-9930aaf04e9f/9fa6cc5e-a76a-4d58-8af7-47af14171882"
-					(reference "#PWR010")
-					(unit 1)
-				)
+					(reference "#PWR099")
+					(unit 1)
+				)

Commit message: OBC: preliminary layout
Parts:
- U4: renamed from U10; symbol 2024-11-27_17-29-01:INA260AIPWR -> INA260AI:INA260AIPWR
- renumbered C17 to C7
Changed lines of the file:
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@@
 		(dnp no)
 		(fields_autoplaced yes)
-		(property "Reference" "C17"
+		(property "Reference" "C7"
 			(at 176.53 106.6864 90)
 			(effects
@@
 			(project "Avionics"
 				(path "/ace5002f-3cbc-4a0a-869b-0e31ebd905b7/893aef5a-59ff-410b-9a71-9930aaf04e9f/740c0668-bfac-47e0-b7b8-de442260ca55"
-					(reference "C17")
+					(reference "C7")
 					(unit 1)
 				)
 				(path "/ace5002f-3cbc-4a0a-869b-0e31ebd905b7/893aef5a-59ff-410b-9a71-9930aaf04e9f/9fa6cc5e-a76a-4d58-8af7-47af14171882"
-					(reference "C24")
+					(reference "C12")
 					(unit 1)
 				)
@@
 		(dnp no)
 		(fields_autoplaced yes)
-		(property "Reference" "#PWR091"
+		(property "Reference" "#PWR046"
 			(at 231.14 152.4 0)
 			(effects
@@
 			(project "Avionics"
 				(path "/ace5002f-3cbc-4a0a-869b-0e31ebd905b7/893aef5a-59ff-410b-9a71-9930aaf04e9f/740c0668-bfac-47e0-b7b8-de442260ca55"
-					(reference "#PWR091")
+					(reference "#PWR046")
 					(unit 1)
 				)
 				(path "/ace5002f-3cbc-4a0a-869b-0e31ebd905b7/893aef5a-59ff-410b-9a71-9930aaf04e9f/9fa6cc5e-a76a-4d58-8af7-47af14171882"
-					(reference "#PWR0100")
+					(reference "#PWR052")
 					(unit 1)
 				)
@@
 	)
 	(symbol
-		(lib_id "2024-11-27_17-29-01:INA260AIPWR")
+		(lib_id "INA260AI:INA260AIPWR")
 		(at 212.09 129.54 0)
 		(unit 1)
@@
 		(dnp no)
 		(fields_autoplaced yes)
-		(property "Reference" "U10"
+		(property "Reference" "U4"
 			(at 212.09 104.14 0)
 			(effects
@@
 			(project "Avionics"
 				(path "/ace5002f-3cbc-4a0a-869b-0e31ebd905b7/893aef5a-59ff-410b-9a71-9930aaf04e9f/740c0668-bfac-47e0-b7b8-de442260ca55"
-					(reference "U10")
+					(reference "U4")
 					(unit 1)
 				)
 				(path "/ace5002f-3cbc-4a0a-869b-0e31ebd905b7/893aef5a-59ff-410b-9a71-9930aaf04e9f/9fa6cc5e-a76a-4d58-8af7-47af14171882"
-					(reference "U13")
+					(reference "U6")
 					(unit 1)
 				)
@@
 		(dnp no)
 		(fields_autoplaced yes)
-		(property "Reference" "#PWR090"
+		(property "Reference" "#PWR045"
 			(at 182.88 93.98 0)
 			(effects
@@
 			(project "Avionics"
 				(path "/ace5002f-3cbc-4a0a-869b-0e31ebd905b7/893aef5a-59ff-410b-9a71-9930aaf04e9f/740c0668-bfac-47e0-b7b8-de442260ca55"
-					(reference "#PWR090")
+					(reference "#PWR045")
 					(unit 1)
 				)
 				(path "/ace5002f-3cbc-4a0a-869b-0e31ebd905b7/893aef5a-59ff-410b-9a71-9930aaf04e9f/9fa6cc5e-a76a-4d58-8af7-47af14171882"
-					(reference "#PWR099")
-					(unit 1)
-				)
+					(reference "#PWR051")
+					(unit 1)
+				)

Commit message: OBC: start PCB layout
Parts:
- renumbered U4 to U3
Changed lines of the file:
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@@
+	)
+	(junction
+		(at 193.04 137.16)
+		(diameter 0)
+		(color 0 0 0 0)
 	)
 	(junction
@@
 	)
 	(junction
-		(at 182.88 137.16)
-		(diameter 0)
-		(color 0 0 0 0)
-	)
-	(junction
 		(at 231.14 144.78)
 		(diameter 0)
@@
 	(wire
 		(pts
-			(xy 182.88 139.7) (xy 182.88 137.16)
+			(xy 193.04 139.7) (xy 193.04 137.16)
 		)
 		(stroke
@@
 	(wire
 		(pts
-			(xy 194.31 139.7) (xy 182.88 139.7)
+			(xy 194.31 139.7) (xy 193.04 139.7)
 		)
 		(stroke
@@
 	(wire
 		(pts
-			(xy 181.61 137.16) (xy 182.88 137.16)
-		)
-		(stroke
-			(width 0)
-			(type default)
-		)
-	)
-	(wire
-		(pts
 			(xy 194.31 119.38) (xy 182.88 119.38)
 		)
@@
 	(wire
 		(pts
-			(xy 182.88 134.62) (xy 182.88 137.16)
+			(xy 193.04 137.16) (xy 194.31 137.16)
+		)
+		(stroke
+			(width 0)
+			(type default)
+		)
+	)
+	(wire
+		(pts
+			(xy 193.04 134.62) (xy 193.04 137.16)
+		)
+		(stroke
+			(width 0)
+			(type default)
+		)
+	)
+	(wire
+		(pts
+			(xy 191.77 137.16) (xy 193.04 137.16)
 		)
 		(stroke
@@
 	(wire
 		(pts
-			(xy 182.88 137.16) (xy 194.31 137.16)
-		)
-		(stroke
-			(width 0)
-			(type default)
-		)
-	)
-	(wire
-		(pts
 			(xy 229.87 119.38) (xy 231.14 119.38)
 		)
@@
 	(wire
 		(pts
-			(xy 194.31 134.62) (xy 182.88 134.62)
+			(xy 194.31 134.62) (xy 193.04 134.62)
 		)
 		(stroke
@@
 	(hierarchical_label "LOAD"
 		(shape output)
-		(at 181.61 137.16 180)
+		(at 191.77 137.16 180)
 		(effects
 			(font
@@
 		(dnp no)
 		(fields_autoplaced yes)
-		(property "Reference" "#PWR046"
+		(property "Reference" "#PWR047"
 			(at 231.14 152.4 0)
 			(effects
@@
 			(project "Avionics"
 				(path "/ace5002f-3cbc-4a0a-869b-0e31ebd905b7/893aef5a-59ff-410b-9a71-9930aaf04e9f/740c0668-bfac-47e0-b7b8-de442260ca55"
-					(reference "#PWR046")
+					(reference "#PWR047")
 					(unit 1)
 				)
 				(path "/ace5002f-3cbc-4a0a-869b-0e31ebd905b7/893aef5a-59ff-410b-9a71-9930aaf04e9f/9fa6cc5e-a76a-4d58-8af7-47af14171882"
-					(reference "#PWR052")
+					(reference "#PWR053")
 					(unit 1)
 				)
@@
 		(dnp no)
 		(fields_autoplaced yes)
-		(property "Reference" "U4"
+		(property "Reference" "U3"
 			(at 212.09 104.14 0)
 			(effects
@@
 			(project "Avionics"
 				(path "/ace5002f-3cbc-4a0a-869b-0e31ebd905b7/893aef5a-59ff-410b-9a71-9930aaf04e9f/740c0668-bfac-47e0-b7b8-de442260ca55"
-					(reference "U4")
+					(reference "U3")
 					(unit 1)
 				)
 				(path "/ace5002f-3cbc-4a0a-869b-0e31ebd905b7/893aef5a-59ff-410b-9a71-9930aaf04e9f/9fa6cc5e-a76a-4d58-8af7-47af14171882"
-					(reference "U6")
+					(reference "U5")
 					(unit 1)
 				)
@@
 		(dnp no)
 		(fields_autoplaced yes)
-		(property "Reference" "#PWR045"
+		(property "Reference" "#PWR046"
 			(at 182.88 93.98 0)
 			(effects
@@
 			(project "Avionics"
 				(path "/ace5002f-3cbc-4a0a-869b-0e31ebd905b7/893aef5a-59ff-410b-9a71-9930aaf04e9f/740c0668-bfac-47e0-b7b8-de442260ca55"
-					(reference "#PWR045")
+					(reference "#PWR046")
 					(unit 1)
 				)
 				(path "/ace5002f-3cbc-4a0a-869b-0e31ebd905b7/893aef5a-59ff-410b-9a71-9930aaf04e9f/9fa6cc5e-a76a-4d58-8af7-47af14171882"
-					(reference "#PWR051")
-					(unit 1)
-				)
+					(reference "#PWR052")
+					(unit 1)
+				)

Commit message: OBC: Continue PCB lauout
Parts:
- renumbered C7 to C3, U3 to U2
Changed lines of the file:
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@@
 		(dnp no)
 		(fields_autoplaced yes)
-		(property "Reference" "C7"
+		(property "Reference" "C3"
 			(at 176.53 106.6864 90)
 			(effects
@@
 		(property "JLCPCB Part Number" "C2649536"
 			(at 182.88 106.68 0)
+			(effects
+				(font
+					(size 1.27 1.27)
+				)
+				(hide yes)
+			)
+		)
+		(property "Field8" ""
+			(at 182.88 106.68 90)
 			(effects
 				(font
@@
 			(project "Avionics"
 				(path "/ace5002f-3cbc-4a0a-869b-0e31ebd905b7/893aef5a-59ff-410b-9a71-9930aaf04e9f/740c0668-bfac-47e0-b7b8-de442260ca55"
-					(reference "C7")
+					(reference "C3")
 					(unit 1)
 				)
 				(path "/ace5002f-3cbc-4a0a-869b-0e31ebd905b7/893aef5a-59ff-410b-9a71-9930aaf04e9f/9fa6cc5e-a76a-4d58-8af7-47af14171882"
-					(reference "C12")
+					(reference "C8")
 					(unit 1)
 				)
@@
 		(dnp no)
 		(fields_autoplaced yes)
-		(property "Reference" "#PWR047"
+		(property "Reference" "#PWR061"
 			(at 231.14 152.4 0)
 			(effects
@@
 			(project "Avionics"
 				(path "/ace5002f-3cbc-4a0a-869b-0e31ebd905b7/893aef5a-59ff-410b-9a71-9930aaf04e9f/740c0668-bfac-47e0-b7b8-de442260ca55"
-					(reference "#PWR047")
+					(reference "#PWR061")
 					(unit 1)
 				)
 				(path "/ace5002f-3cbc-4a0a-869b-0e31ebd905b7/893aef5a-59ff-410b-9a71-9930aaf04e9f/9fa6cc5e-a76a-4d58-8af7-47af14171882"
-					(reference "#PWR053")
+					(reference "#PWR067")
 					(unit 1)
 				)
@@
 		(dnp no)
 		(fields_autoplaced yes)
-		(property "Reference" "U3"
+		(property "Reference" "U2"
 			(at 212.09 104.14 0)
 			(effects
@@
 		)
 		(property "JLCPCB Part Number" "C2155885"
+			(at 212.09 129.54 0)
+			(effects
+				(font
+					(size 1.27 1.27)
+				)
+				(hide yes)
+			)
+		)
+		(property "Field8" ""
 			(at 212.09 129.54 0)
 			(effects
@@
 			(project "Avionics"
 				(path "/ace5002f-3cbc-4a0a-869b-0e31ebd905b7/893aef5a-59ff-410b-9a71-9930aaf04e9f/740c0668-bfac-47e0-b7b8-de442260ca55"
-					(reference "U3")
+					(reference "U2")
 					(unit 1)
 				)
 				(path "/ace5002f-3cbc-4a0a-869b-0e31ebd905b7/893aef5a-59ff-410b-9a71-9930aaf04e9f/9fa6cc5e-a76a-4d58-8af7-47af14171882"
-					(reference "U5")
+					(reference "U4")
 					(unit 1)
 				)
@@
 		(dnp no)
 		(fields_autoplaced yes)
-		(property "Reference" "#PWR046"
+		(property "Reference" "#PWR060"
 			(at 182.88 93.98 0)
 			(effects
@@
 			(project "Avionics"
 				(path "/ace5002f-3cbc-4a0a-869b-0e31ebd905b7/893aef5a-59ff-410b-9a71-9930aaf04e9f/740c0668-bfac-47e0-b7b8-de442260ca55"
-					(reference "#PWR046")
+					(reference "#PWR060")
 					(unit 1)
 				)
 				(path "/ace5002f-3cbc-4a0a-869b-0e31ebd905b7/893aef5a-59ff-410b-9a71-9930aaf04e9f/9fa6cc5e-a76a-4d58-8af7-47af14171882"
-					(reference "#PWR052")
-					(unit 1)
-				)
+					(reference "#PWR066")
+					(unit 1)
+				)

Commit message: Layout confirmed, PCBs ordered
Parts:
- C3: DigiKey Part Number 399-C0603C104M5RACTUCT-ND -> 720-GA0805Y104JXABT31GCT-ND
Changed lines of the file:
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@@
 			)
 		)
-		(property "DigiKey Part Number" "399-C0603C104M5RACTUCT-ND"
+		(property "DigiKey Part Number" "720-GA0805Y104JXABT31GCT-ND"
 			(at 182.88 106.68 0)
 			(effects
@@
 			)
 		)
-		(property "Datasheet" "INA260AIPWR"
+		(property "Datasheet" ""
 			(at 212.09 129.54 0)
 			(effects
