File: TPS543320.kicad_sch (KiCad schematic)
At the start: 19 parts, among them U5 TPS543320RPYR

Commit message: Separate PCBs into individual repos to allow for multiple workgroups
Other:
- title: HEDGE2 Avionics -> HEDGE2 OBC
Changed lines of the file:
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@@
 	(paper "USLedger")
 	(title_block
-		(title "HEDGE2 Avionics")
+		(title "HEDGE2 OBC")
 		(date "2025-06-27")
 		(rev "V0.8")
@@
 		)
 		(instances
-			(project "Avionics"
+			(project "HEDGE2-OBC"
 				(path "/ace5002f-3cbc-4a0a-869b-0e31ebd905b7/893aef5a-59ff-410b-9a71-9930aaf04e9f/e2cad078-3ca5-46c7-a65f-c1e6fb9d60cb"
 					(reference "#PWR074")
@@
 		)
 		(instances
-			(project "Avionics"
+			(project "HEDGE2-OBC"
 				(path "/ace5002f-3cbc-4a0a-869b-0e31ebd905b7/893aef5a-59ff-410b-9a71-9930aaf04e9f/e2cad078-3ca5-46c7-a65f-c1e6fb9d60cb"
 					(reference "#PWR076")
@@
 		)
 		(instances
-			(project "Avionics"
+			(project "HEDGE2-OBC"
 				(path "/ace5002f-3cbc-4a0a-869b-0e31ebd905b7/893aef5a-59ff-410b-9a71-9930aaf04e9f/e2cad078-3ca5-46c7-a65f-c1e6fb9d60cb"
 					(reference "U5")
@@
 		)
 		(instances
-			(project "Avionics"
+			(project "HEDGE2-OBC"
 				(path "/ace5002f-3cbc-4a0a-869b-0e31ebd905b7/893aef5a-59ff-410b-9a71-9930aaf04e9f/e2cad078-3ca5-46c7-a65f-c1e6fb9d60cb"
 					(reference "C16")
