File: rp2040.kicad_sch (KiCad schematic)
At the start: 0 parts

Commit message: Separate PCBs into individual repos to allow for multiple workgroups
Other:
- title: HEDGE2 Avionics -> HEDGE2 OBC
Changed lines of the file:
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@@
 	(paper "USLedger")
 	(title_block
-		(title "HEDGE2 Avionics")
+		(title "HEDGE2 OBC")
 		(date "2025-06-27")
 		(rev "V0.8")
