File: HEDGE2-OBC.kicad_sch (KiCad schematic)
At the start: 27 parts, among them J1 SQT-110-01-L-D, J2 MMBX-S50-0-18, J3 SMA-J-P-X-RA-TH1, U1 OEM719

Commit message: Separate PCBs into individual repos to allow for multiple workgroups
Other:
- title: HEDGE2 Avionics -> HEDGE2 OBC

Commit message: Cleanup after splitting PCBs into separate repos
Parts:
- renumbered Module1 to Module2
Connections:
- net GND: now also Module2.13 (GND), Module2.14 (GND), Module2.19 (Ethernet_nLED1(3.3v)), Module2.20 (EEPROM_nWP), Module2.25 (GPIO21), Module2.26 (GPIO19), Module2.31 (GPIO12), Module2.32 (GND), Module2.37 (GPIO7), Module2.38 (GPIO11), Module2.44 (GPIO10), Module2.50 (GPIO17), Module2.55 (GPIO14), Module2.56 (GPIO3), Module2.61 (SD_DAT3), Module2.62 (SD_CMD), Module2.67 (SD_DAT1), Module2.68 (SD_DAT4), Module2.7 (GND), Module2.73 (SD_VDD_Override), Module2.74 (GND), Module2.79 (+5v_(Input)), Module2.8 (GND), Module2.80 (SCL0), Module2.85 (+5v_(Input)), Module2.86 (+3.3v_(Output)), Module2.91 (BT_nDisable), Module2.92 (RUN_PG), Module2.97 (Camera_GPIO), Module2.98 (GND); no longer Module2.107 (GND), Module2.108 (GND), Module2.113 (GND), Module2.114 (GND), Module2.119 (GND), Module2.120 (GND), Module2.125 (GND), Module2.126 (GND), Module2.131 (GND), Module2.132 (GND), Module2.137 (GND), Module2.138 (GND), Module2.144 (GND), Module2.150 (GND), Module2.155 (GND), Module2.156 (GND), Module2.161 (GND), Module2.162 (GND), Module2.167 (GND), Module2.168 (GND), Module2.173 (GND), Module2.174 (GND), Module2.179 (GND), Module2.180 (GND), Module2.185 (GND), Module2.186 (GND), Module2.191 (GND), Module2.192 (GND), Module2.197 (GND), Module2.198 (GND)
Other:
- removed sheet TPS543320
- title: HEDGE2 OBC -> HEDGE-2 OBC
- moved on the sheet: C1, C2, D1, D2, J1, J2, J3, R1, R2, R3, R4, R5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

Commit message: Add RS-485 interfaces; modify for 5V power input
Parts:
- removed Module1: ComputeModule4, CM4102008:MODULE_CM4102008, symbol CM4IO:ComputeModule4-CM4
- removed U1: OEM719, Novatel:OEM719, symbol HEDGE2:NOVATEL OEM719
- added unit 2 of Module1
- renumbered J2 to J1, J1 to J2, Module2 to Module1, R7 to R5, R8 to R6, R5 to R7, R6 to R8
Connections:
- net +3V3: now also Module1.78 (GPIO_VREF(1.8v/3.3v_Input)), Module1.84 (+3.3v_(Output)), Module1.86 (+3.3v_(Output))
- net +5V_CM4: now also Module1.77 (+5v_(Input)), Module1.79 (+5v_(Input)), Module1.81 (+5v_(Input)), Module1.83 (+5v_(Input)), Module1.85 (+5v_(Input)), Module1.87 (+5v_(Input))
- net +5V_GNSS: no longer H1OBC1.48
- net +5V_MPU: no longer H1OBC1.46
- net CAN_A_RXD: now also Module1.51 (GPIO15)
- net CAN_A_S: now also Module1.29 (GPIO16)
- net CAN_A_TXD: now also Module1.55 (GPIO14)
- net CAN_B_RXD: now also Module1.35 (ID_SC)
- net CAN_B_S: now also Module1.58 (GPIO2)
- net CAN_B_TXD: now also Module1.36 (ID_SD)
- net GND: now also Module1.1 (GND), Module1.2 (GND), Module1.22 (GND), Module1.23 (GND), Module1.33 (GND), Module1.42 (GND), Module1.43 (GND), Module1.52 (GND), Module1.53 (GND), Module1.59 (GND), Module1.60 (GND), Module1.65 (GND), Module1.66 (GND), Module1.71 (GND), Module1.107 (GND), Module1.108 (GND), Module1.113 (GND), Module1.114 (GND), Module1.119 (GND), Module1.120 (GND), Module1.125 (GND), Module1.126 (GND), Module1.131 (GND), Module1.132 (GND), Module1.137 (GND), Module1.138 (GND), Module1.144 (GND), Module1.150 (GND), Module1.155 (GND), Module1.156 (GND), Module1.161 (GND), Module1.162 (GND), Module1.167 (GND), Module1.168 (GND), Module1.173 (GND), Module1.174 (GND), Module1.179 (GND), Module1.180 (GND), Module1.185 (GND), Module1.186 (GND), Module1.191 (GND), Module1.192 (GND), Module1.197 (GND), Module1.198 (GND); no longer Module1.19 (Ethernet_nLED1(3.3v)), Module1.20 (EEPROM_nWP), Module1.25 (GPIO21), Module1.26 (GPIO19), Module1.31 (GPIO12), Module1.37 (GPIO7), Module1.38 (GPIO11), Module1.44 (GPIO10), Module1.50 (GPIO17), Module1.55 (GPIO14), Module1.56 (GPIO3), Module1.61 (SD_DAT3), Module1.62 (SD_CMD), Module1.67 (SD_DAT1), Module1.68 (SD_DAT4), Module1.73 (SD_VDD_Override), Module1.79 (+5v_(Input)), Module1.80 (SCL0), Module1.85 (+5v_(Input)), Module1.86 (+3.3v_(Output)), Module1.91 (BT_nDisable), Module1.92 (RUN_PG), Module1.97 (Camera_GPIO)
- net GNSS_NRESET_IN: now also Module1.38 (GPIO11)
- net GNSS_PPS: now also Module1.46 (GPIO22)
- net GNSS_PV: now also Module1.50 (GPIO17)
- net GNSS_RXD1: no longer H1OBC1.44
- net GNSS_RXD2: now also Module1.34 (GPIO5)
- net GNSS_TXD1: no longer H1OBC1.42
- net GNSS_TXD2: now also Module1.54 (GPIO4)
- net PI_nLED_Activity: now also Module1.21 (PI_nLED_Activity)
- net SCL0: now also Module1.80 (SCL0)
- net SDA0: now also Module1.82 (SDA0)
- net UART_COMM_RX: now also Module1.40 (GPIO9); no longer H1OBC1.24
- net UART_COMM_TX: now also Module1.39 (GPIO8); no longer H1OBC1.22
- net nPWR_LED: now also Module1.95 (nPI_LED_PWR)
- net UART_SCI_RX: now reaches Module1.28 (GPIO13)
- net at Module1.89 (WiFi_nDisable): now also R5.2
- net at R6.1: now also Module1.91 (BT_nDisable)
- net UART_DATA_RX renamed UART_E_RX
- net UART_DATA_TX renamed UART_E_TX
- new net PWR_1: H1OBC1.46
- new net PWR_2: H1OBC1.48
- new net UART_D_RX: H1OBC1.24
- new net UART_D_TX: H1OBC1.22
- new net UART_F_RX: H1OBC1.44
- new net UART_F_TX: H1OBC1.42
- new net UART_SCI_TX: Module1.31 (GPIO12)
- no-connect marks 214 -> 207
Other:
- added sheet SN65HVD1782 (SN65HVD1782.kicad_sch)
- added sheet SN65HVD1783 (SN65HVD1782.kicad_sch)
- note removed: "CM4 UART4"
- note removed: "CM4 UART5"
- note removed: "OEM719B UART1 (CONFIG)"
- note removed: "SPACECRAFT BUS CONNECTIONS"
- moved on the sheet: C1, C2, J1, J2, J3, Module1A, R1, R2, R3, R4
